File: ESP32Webradio_5.kicad_pcb (KiCad board)
At the start: 2 copper layers, 44 x 54 mm, 17 parts, among them J1 5V, J2 Rotary Encoder, J3 Display, J5 SJ1-3523N, U1 esp32_38_pins-custom_library

Commit message: corrigate restor values
Parts:
- R1: value 100k -> 10k
- R2, R5: value 47k -> 4.7k
- R3, R4: value 2.2k -> 22k
Changed lines of the file:
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@@
       (effects (font (size 1 1) (thickness 0.15)))
     )
-    (fp_text value "47k" (at 2.032 1.905 90) (layer "F.Fab")
+    (fp_text value "4.7k" (at 2.032 1.905 90) (layer "F.Fab")
       (effects (font (size 1 1) (thickness 0.15)))
     )
@@
       (effects (font (size 1 1) (thickness 0.15)))
     )
-    (fp_text value "47k" (at 8.12 2.228 -90) (layer "F.Fab")
+    (fp_text value "4.7k" (at 8.12 2.228 -90) (layer "F.Fab")
       (effects (font (size 1 1) (thickness 0.15)))
     )
@@
       (effects (font (size 1 1) (thickness 0.15)))
     )
-    (fp_text value "2.2k" (at 0.762 2.032 90) (layer "F.Fab")
+    (fp_text value "22k" (at 0.762 2.032 90) (layer "F.Fab")
       (effects (font (size 1 1) (thickness 0.15)))
     )
@@
       (effects (font (size 1 1) (thickness 0.15)))
     )
-    (fp_text value "100k" (at 5.06 1.7 -90) (layer "F.Fab")
+    (fp_text value "10k" (at 5.06 1.7 -90) (layer "F.Fab")
       (effects (font (size 1 1) (thickness 0.15)))
     )
@@
       (effects (font (size 1 1) (thickness 0.15)))
     )
-    (fp_text value "2.2k" (at 1.143 2.032 90) (layer "F.Fab")
+    (fp_text value "22k" (at 1.143 2.032 90) (layer "F.Fab")
       (effects (font (size 1 1) (thickness 0.15)))
     )
@@
       (effects (font (size 1.000402 1.000402) (thickness 0.15)))
     )
-    (fp_text value "SJ1-3523N" (at 2.46 7.7945 90) (layer "F.Fab")
+    (fp_text value "SJ1-3523N" (at 4.75889 7.64126 90) (layer "F.Fab")
       (effects (font (size 1.000819 1.000819) (thickness 0.15)))
     )
-    (fp_text user "PCB-edge" (at -0.59 -2.6555 90) (layer "Dwgs.User")
+    (fp_text user "PCB-edge" (at -12.5245 -6.01177 90) (layer "Dwgs.User")
       (effects (font (size 0.801567 0.801567) (thickness 0.15)))
     )
-    (fp_line (start -3.5 -4.5) (end -4.3 -4.5) (layer "F.SilkS") (width 0.127))
     (fp_line (start 7.5 6.2) (end -3.5 6.2) (layer "F.SilkS") (width 0.127))
     (fp_line (start -3.5 4.5) (end -4.3 4.5) (layer "F.SilkS") (width 0.127))
+    (fp_line (start 7.5 -6.2) (end -3.5 -6.2) (layer "F.SilkS") (width 0.127))
     (fp_line (start -3.5 4.5) (end -3.5 6.2) (layer "F.SilkS") (width 0.127))
-    (fp_line (start 7.5 -6.2) (end -3.5 -6.2) (layer "F.SilkS") (width 0.127))
     (fp_line (start -3.5 -6.2) (end -3.5 -4.5) (layer "F.SilkS") (width 0.127))
     (fp_line (start 7.5 -6.2) (end 7.5 6.2) (layer "F.SilkS") (width 0.127))
+    (fp_line (start -3.5 -4.5) (end -4.3 -4.5) (layer "F.SilkS") (width 0.127))
     (fp_circle (center 0 -6.8) (end 0.17 -6.8) (layer "F.SilkS") (width 0.34) (fill none))
     (fp_line (start 7.75 -6.45) (end 7.75 6.45) (layer "F.CrtYd") (width 0.05))
+    (fp_line (start -6.75 -3.25) (end -6.75 3.25) (layer "F.CrtYd") (width 0.05))
     (fp_line (start -4.75 -6.45) (end 7.75 -6.45) (layer "F.CrtYd") (width 0.05))
+    (fp_line (start -4.75 3.25) (end -4.75 6.45) (layer "F.CrtYd") (width 0.05))
     (fp_line (start 7.75 6.45) (end -4.75 6.45) (layer "F.CrtYd") (width 0.05))
-    (fp_line (start -6.75 -3.25) (end -6.75 3.25) (layer "F.CrtYd") (width 0.05))
-    (fp_line (start -4.75 3.25) (end -4.75 6.45) (layer "F.CrtYd") (width 0.05))
     (fp_line (start -4.75 -3.25) (end -6.75 -3.25) (layer "F.CrtYd") (width 0.05))
     (fp_line (start -4.75 -6.45) (end -4.75 -3.25) (layer "F.CrtYd") (width 0.05))
     (fp_line (start -6.75 3.25) (end -4.75 3.25) (layer "F.CrtYd") (width 0.05))
-    (fp_line (start -6.5 -3) (end -6.5 3) (layer "F.Fab") (width 0.127))
-    (fp_line (start 7.5 6.2) (end -3.5 6.2) (layer "F.Fab") (width 0.127))
-    (fp_line (start -4.5 4.5) (end -3.5 4.5) (layer "F.Fab") (width 0.127))
+    (fp_line (start 7.5 -6.2) (end -3.5 -6.2) (layer "F.Fab") (width 0.127))
     (fp_line (start -3.5 -6.2) (end -3.5 -4.5) (layer "F.Fab") (width 0.127))
     (fp_line (start -3.5 -4.5) (end -4.5 -4.5) (layer "F.Fab") (width 0.127))
+    (fp_line (start -4.5 -3) (end -4.5 3) (layer "F.Fab") (width 0.127))
     (fp_line (start -3.5 4.5) (end -3.5 6.2) (layer "F.Fab") (width 0.127))
+    (fp_line (start -6.5 -3) (end -6.5 3) (layer "F.Fab") (width 0.127))
     (fp_line (start -4.5 -3) (end -6.5 -3) (layer "F.Fab") (width 0.127))
+    (fp_line (start -4.5 3) (end -4.5 4.5) (layer "F.Fab") (width 0.127))
+    (fp_line (start 7.5 6.2) (end -3.5 6.2) (layer "F.Fab") (width 0.127))
+    (fp_line (start -4.5 -4.5) (end -4.5 -3) (layer "F.Fab") (width 0.127))
     (fp_line (start 7.5 -6.2) (end 7.5 6.2) (layer "F.Fab") (width 0.127))
-    (fp_line (start 7.5 -6.2) (end -3.5 -6.2) (layer "F.Fab") (width 0.127))
-    (fp_line (start -4.5 3) (end -4.5 4.5) (layer "F.Fab") (width 0.127))
     (fp_line (start -6.5 3) (end -4.5 3) (layer "F.Fab") (width 0.127))
-    (fp_line (start -4.5 -3) (end -4.5 3) (layer "F.Fab") (width 0.127))
-    (fp_line (start -4.5 -4.5) (end -4.5 -3) (layer "F.Fab") (width 0.127))
+    (fp_line (start -4.5 4.5) (end -3.5 4.5) (layer "F.Fab") (width 0.127))
+    (pad "" np_thru_hole circle (at 5 0 90) (size 1.2 1.2) (drill 1.2) (layers *.Cu *.Mask))
+    (pad "" np_thru_hole circle (at 0 5 90) (size 1.2 1.2) (drill 1.2) (layers *.Cu *.Mask))
     (pad "" np_thru_hole circle (at 0 -5 90) (size 1.2 1.2) (drill 1.2) (layers *.Cu *.Mask))
+    (pad "" np_thru_hole circle (at -2.5 -5 90) (size 1.2 1.2) (drill 1.2) (layers *.Cu *.Mask))
     (pad "" np_thru_hole circle (at -2.5 5 90) (size 1.2 1.2) (drill 1.2) (layers *.Cu *.Mask))
-    (pad "" np_thru_hole circle (at 0 5 90) (size 1.2 1.2) (drill 1.2) (layers *.Cu *.Mask))
-    (pad "" np_thru_hole circle (at 5 0 90) (size 1.2 1.2) (drill 1.2) (layers *.Cu *.Mask))
-    (pad "" np_thru_hole circle (at -2.5 -5 90) (size 1.2 1.2) (drill 1.2) (layers *.Cu *.Mask))
     (pad "1" thru_hole oval (at 0 0 90) (size 1.308 2.616) (drill oval 0.8 1.5) (layers *.Cu *.Mask)
       (net 5 "GND") (pintype "passive"))
+    (pad "2" thru_hole oval (at 5 5 90) (size 2.616 1.308) (drill oval 1.5 0.8) (layers *.Cu *.Mask)
+      (net 41 "/S") (pintype "passive"))
     (pad "2" thru_hole oval (at 5.075389 2.532895 90) (size 2.616 1.308) (drill oval 1.5 0.8) (layers *.Cu *.Mask)
       (net 41 "/S") (pintype "passive"))
-    (pad "2" thru_hole oval (at 5 5 90) (size 2.616 1.308) (drill oval 1.5 0.8) (layers *.Cu *.Mask)
-      (net 41 "/S") (pintype "passive"))
     (pad "3" thru_hole oval (at 5.08 -2.54 90) (size 2.616 1.308) (drill oval 1.5 0.8) (layers *.Cu *.Mask)
