File: ESP32Webradio_5.kicad_sch (KiCad schematic)
At the start: 17 parts, among them J1 5V, J2 Rotary Encoder, J3 Display, J5 SJ1-3523N, U1 esp32_38_pins-custom_library

Commit message: corrigate restor values
Parts:
- R1: value 100k -> 10k
- R2, R5: value 47k -> 4.7k
- R3, R4: value 2.2k -> 22k
Changed lines of the file:
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@@
     (in_bom yes) (on_board yes) (fields_autoplaced)
     (property "Reference" "R3" (id 0) (at 186.69 127 90))
-    (property "Value" "2.2k" (id 1) (at 186.69 129.54 90))
+    (property "Value" "22k" (id 1) (at 186.69 129.54 90))
     (property "Footprint" "Resistor_THT:R_Axial_DIN0204_L3.6mm_D1.6mm_P7.62mm_Horizontal" (id 2) (at 186.69 135.128 90)
       (effects (font (size 1.27 1.27)) hide)
@@
     (in_bom yes) (on_board yes) (fields_autoplaced)
     (property "Reference" "R4" (id 0) (at 186.69 137.16 90))
-    (property "Value" "2.2k" (id 1) (at 186.69 139.7 90))
+    (property "Value" "22k" (id 1) (at 186.69 139.7 90))
     (property "Footprint" "Resistor_THT:R_Axial_DIN0204_L3.6mm_D1.6mm_P7.62mm_Horizontal" (id 2) (at 186.69 145.288 90)
       (effects (font (size 1.27 1.27)) hide)
@@
       (effects (font (size 1.27 1.27)) (justify left))
     )
-    (property "Value" "100k" (id 1) (at 88.9 47.6249 0)
+    (property "Value" "10k" (id 1) (at 88.9 47.6249 0)
       (effects (font (size 1.27 1.27)) (justify left))
     )
@@
     (in_bom yes) (on_board yes) (fields_autoplaced)
     (property "Reference" "R5" (id 0) (at 161.925 137.16 90))
-    (property "Value" "47k" (id 1) (at 161.925 139.7 90))
+    (property "Value" "4.7k" (id 1) (at 161.925 139.7 90))
     (property "Footprint" "Resistor_THT:R_Axial_DIN0204_L3.6mm_D1.6mm_P7.62mm_Horizontal" (id 2) (at 161.925 145.288 90)
       (effects (font (size 1.27 1.27)) hide)
@@
     (in_bom yes) (on_board yes) (fields_autoplaced)
     (property "Reference" "R2" (id 0) (at 161.925 127 90))
-    (property "Value" "47k" (id 1) (at 161.925 129.54 90))
+    (property "Value" "4.7k" (id 1) (at 161.925 129.54 90))
     (property "Footprint" "Resistor_THT:R_Axial_DIN0204_L3.6mm_D1.6mm_P7.62mm_Horizontal" (id 2) (at 161.925 135.128 90)
       (effects (font (size 1.27 1.27)) hide)
@@
     )
     (path "/8cf50433-5d1e-4e8e-a26a-2df3e5bda93c"
-      (reference "R1") (unit 1) (value "100k") (footprint "Resistor_THT:R_Axial_DIN0204_L3.6mm_D1.6mm_P7.62mm_Horizontal")
+      (reference "R1") (unit 1) (value "10k") (footprint "Resistor_THT:R_Axial_DIN0204_L3.6mm_D1.6mm_P7.62mm_Horizontal")
     )
     (path "/daeaf536-deaf-44e0-9971-669bd8f53219"
-      (reference "R2") (unit 1) (value "47k") (footprint "Resistor_THT:R_Axial_DIN0204_L3.6mm_D1.6mm_P7.62mm_Horizontal")
+      (reference "R2") (unit 1) (value "4.7k") (footprint "Resistor_THT:R_Axial_DIN0204_L3.6mm_D1.6mm_P7.62mm_Horizontal")
     )
     (path "/04d45744-33cf-4f4b-8d27-accce5a435a4"
-      (reference "R3") (unit 1) (value "2.2k") (footprint "Resistor_THT:R_Axial_DIN0204_L3.6mm_D1.6mm_P7.62mm_Horizontal")
+      (reference "R3") (unit 1) (value "22k") (footprint "Resistor_THT:R_Axial_DIN0204_L3.6mm_D1.6mm_P7.62mm_Horizontal")
     )
     (path "/209892e6-d1c6-4d50-89bc-859917e3a84d"
-      (reference "R4") (unit 1) (value "2.2k") (footprint "Resistor_THT:R_Axial_DIN0204_L3.6mm_D1.6mm_P7.62mm_Horizontal")
+      (reference "R4") (unit 1) (value "22k") (footprint "Resistor_THT:R_Axial_DIN0204_L3.6mm_D1.6mm_P7.62mm_Horizontal")
     )
     (path "/97bfa3b2-22c2-4840-80e3-41afd38dd7c9"
-      (reference "R5") (unit 1) (value "47k") (footprint "Resistor_THT:R_Axial_DIN0204_L3.6mm_D1.6mm_P7.62mm_Horizontal")
+      (reference "R5") (unit 1) (value "4.7k") (footprint "Resistor_THT:R_Axial_DIN0204_L3.6mm_D1.6mm_P7.62mm_Horizontal")
     )
     (path "/efb6a8e5-cd95-40c8-95e3-2301d961f4a9"
